Commit message: done with testing sensors and implementing SLAM and Navigation

File: description/gazebo_control.xacro (robot description, xacro)
@@ -5,6 +5,6 @@
             <left_joint>left_wheel_joint</left_joint>
             <right_joint>right_wheel_joint</right_joint>
-            <wheel_separation>0.35</wheel_separation>
-            <wheel_diameter>0.1</wheel_diameter>
+            <wheel_separation>0.55</wheel_separation>
+            <wheel_diameter>0.16</wheel_diameter>
             <max_wheel_torque>20.0</max_wheel_torque>
             <max_wheel_acceleration>10.0</max_wheel_acceleration>

File: description/lidar.xacro (robot description, xacro)
@@ -30,6 +30,6 @@
         <sensor name="lidar" type="ray">
             <pose>0 0 0 0 0 0</pose>
-            <always_on>false</always_on>
-            <visualize>false</visualize>
+            <always_on>true</always_on>
+            <visualize>true</visualize>
             <update_rate>10</update_rate>
             <ray>

File: description/robot.urdf.xacro (robot description, xacro)
@@ -4,4 +4,5 @@
     <xacro:include filename="gazebo_control.xacro" />
     <xacro:include filename="lidar.xacro" />
-    <xacro:include filename="camera.xacro" />
+   <!-- <xacro:include filename="camera.xacro" /> -->
+    <xacro:include filename="depth_camera.xacro" />
 </robot>

File: description/robot_core.xacro (robot description, xacro)
@@ -25,5 +25,5 @@
                 <box size="0.5 0.5 0.2"/>
             </geometry>
-            <material name="orange"/>
+            <material name="red"/>
         </visual>
         <collision>
@@ -66,5 +66,5 @@
                 <cylinder radius="0.08" length="0.05"/>
             </geometry>
-            <material name="black"/>
+            <material name="blue"/>
         </visual>
         <collision>
@@ -93,5 +93,5 @@
         <parent link="base_link"/>
         <child link="right_wheel"/>
-        <origin xyz="0 -0.275 0" rpy="1.5708 0 0"/>
+        <origin xyz="0 -0.275 0" rpy="-1.5708 0 0"/>
         <axis xyz="0 0 1"/>
     </joint>
@@ -102,5 +102,5 @@
                 <cylinder radius="0.08" length="0.05"/>
             </geometry>
-            <material name="black"/>
+            <material name="blue"/>
         </visual>
         <collision>
@@ -137,5 +137,5 @@
                 <sphere radius="0.08"/>
             </geometry>
-            <material name="red"/>
+            <material name="black"/>
         </visual>
         <collision>
@@ -159,6 +159,6 @@
     <gazebo reference="caster_wheel">
         <material>Gazebo/Black</material>
-        <mu1 value="0.001"/>
-        <mu2 value="0.001"/>
+        <mu1 value="0.1"/>
+        <mu2 value="0.1"/>
     </gazebo>
 </robot>
